Commit message: version hongo_aero

File: rotors_description/urdf/component_snippets.xacro (robot description, xacro)
@@ -554,5 +554,5 @@
   <!-- Macro to add a VI-sensor camera. -->
   <xacro:macro name="vi_sensor_camera_macro"
-    params="namespace parent_link camera_suffix frame_rate *origin">
+    params="namespace parent_link camera_suffix frame_rate horizontal_fov *origin">
     <xacro:camera_macro
       namespace="${namespace}"
@@ -560,5 +560,5 @@
       camera_suffix="${camera_suffix}"
       frame_rate="${frame_rate}"
-      horizontal_fov="1.3962634"
+      horizontal_fov="${horizontal_fov}"
       image_width="752"
       image_height="480"
@@ -575,5 +575,5 @@
   <!-- Macro to add a VI-sensor stereo camera. -->
   <xacro:macro name="vi_sensor_stereo_camera_macro"
-    params="namespace parent_link frame_rate origin_offset_x baseline_y origin_offset_z max_range">
+    params="namespace parent_link frame_rate origin_offset_x baseline_y origin_offset_z max_range horizontal_fov">
     <xacro:stereo_camera_macro
       namespace="${namespace}"
@@ -581,5 +581,5 @@
       parent_link="${parent_link}"
       frame_rate="${frame_rate}"
-      horizontal_fov="1.3962634"
+      horizontal_fov="${horizontal_fov}"
       image_width="752"
       image_height="480"
@@ -598,5 +598,5 @@
   <!-- Macro to add a depth camera on the VI-sensor. -->
   <xacro:macro name="vi_sensor_depth_macro"
-    params="namespace parent_link camera_suffix frame_rate max_range *origin">
+    params="namespace parent_link camera_suffix frame_rate max_range horizontal_fov *origin">
     <link name="${namespace}/camera_${camera_suffix}_link">
       <collision>
@@ -631,5 +631,5 @@
         <update_rate>${frame_rate}</update_rate>
         <camera>
-          <horizontal_fov>2</horizontal_fov>
+          <horizontal_fov>${horizontal_fov}</horizontal_fov>
           <image>
             <format>L8</format>
@@ -666,5 +666,5 @@
   </xacro:macro>
   <!-- VI-Sensor Macro -->
-  <xacro:macro name="vi_sensor_macro" params="namespace parent_link enable_cameras enable_depth enable_ground_truth *origin">
+  <xacro:macro name="vi_sensor_macro" params="namespace parent_link enable_cameras enable_depth enable_ground_truth horizontal_fov *origin">
     <!-- Vi Sensor Link -->
     <link name="${namespace}/vi_sensor_link">
@@ -682,5 +682,5 @@
       </visual>
       <inertial>
-        <mass value="0.13" />
+        <mass value="1e-6" />
         <origin xyz="0 0 0" rpy="0 0 0" />
         <inertia ixx="1e-6" ixy="0" ixz="0" iyy="1e-6" iyz="0" izz="1e-6" />
@@ -698,5 +698,5 @@
         namespace="${namespace}" parent_link="${namespace}/vi_sensor_link"
         frame_rate="30.0" origin_offset_x="0.015" baseline_y="${0.055*2}"
-        origin_offset_z="0.0065" max_range="30.0">
+        origin_offset_z="0.0065" max_range="30.0" horizontal_fov="${horizontal_fov}">
       </xacro:vi_sensor_stereo_camera_macro>
     </xacro:if>
@@ -705,5 +705,5 @@
       <xacro:vi_sensor_depth_macro
         namespace="${namespace}" parent_link="${namespace}/vi_sensor_link"
-        camera_suffix="depth" frame_rate="30.0" max_range="10.0">
+        camera_suffix="depth" frame_rate="30.0" max_range="10.0" horizontal_fov="${horizontal_fov}">
         <origin xyz="0.015 0.055 0.0065" rpy="0 0 0" />
       </xacro:vi_sensor_depth_macro>

File: rotors_description/urdf/firefly_base.xacro (robot description, xacro)
@@ -17,4 +17,14 @@
 -->
 <robot name="firefly" xmlns:xacro="http://ros.org/wiki/xacro">
+  <!-- hokuyo 2d lidar -->
+  <xacro:include filename="$(find rotors_description)/urdf/hokuyo.urdf.xacro"/>
+  <xacro:if value="$(arg 1DoF_gimbal)">
+      <!-- 1dof gimbal -->
+      <xacro:include filename="$(find rotors_description)/urdf/1Dof_gimbal.urdf.xacro"/>
+  </xacro:if>
+  <xacro:if value="$(arg 3DoF_gimbal)">
+      <!-- 3dof gimbal -->
+      <xacro:include filename="$(find rotors_description)/urdf/3Dof_gimbal.urdf.xacro"/>
+  </xacro:if>
   <xacro:include filename="$(find rotors_description)/urdf/component_snippets.xacro" />
   <!-- Instantiate firefly "mechanics" -->
@@ -33,4 +43,18 @@
     <xacro:ground_truth_imu_and_odometry namespace="${namespace}" parent_link="${namespace}/base_link" />
   </xacro:if>
+  <!-- hokuyo 2d lidar -->
+  <sensor_hokuyo parent="${namespace}/base_link"/>
+  <!-- gimbal-->
+  <gimbal namespace="${namespace}" parent="${namespace}/base_link"/>
+  <!-- depth camera-->
+  <vi_sensor_macro
+    namespace="${namespace}/vi_sensor"
+    parent_link="${namespace}/gimbal_arm_end"
+    enable_cameras="true"
+    enable_depth="true"
+    enable_ground_truth="true"
+    horizontal_fov="$(arg horizontal_fov)">
+    <origin xyz="0 0 0" rpy="0.0 0.1 0.0" />
+</vi_sensor_macro>
   <xacro:if value="$(arg enable_logging)">
     <!-- Instantiate a logger -->

Commit message: Enable to control 1 or 3 DoF gimbal

File: rotors_description/urdf/component_snippets.xacro (robot description, xacro)
@@ -575,5 +575,5 @@
   <!-- Macro to add a VI-sensor stereo camera. -->
   <xacro:macro name="vi_sensor_stereo_camera_macro"
-    params="namespace parent_link frame_rate origin_offset_x baseline_y origin_offset_z max_range horizontal_fov">
+    params="namespace parent_link frame_rate origin_offset_x baseline_y origin_offset_z max_range min_range width height horizontal_fov">
     <xacro:stereo_camera_macro
       namespace="${namespace}"
@@ -582,8 +582,8 @@
       frame_rate="${frame_rate}"
       horizontal_fov="${horizontal_fov}"
-      image_width="752"
-      image_height="480"
+      image_width="${width}"
+      image_height="${height}"
       image_format="L8"
-      min_distance="0.02"
+      min_distance="${min_range}"
       max_distance="${max_range}"
       noise_mean="0.0"
@@ -598,5 +598,5 @@
   <!-- Macro to add a depth camera on the VI-sensor. -->
   <xacro:macro name="vi_sensor_depth_macro"
-    params="namespace parent_link camera_suffix frame_rate max_range horizontal_fov *origin">
+    params="namespace parent_link camera_suffix frame_rate min_range max_range width height horizontal_fov *origin">
     <link name="${namespace}/camera_${camera_suffix}_link">
       <collision>
@@ -634,9 +634,9 @@
           <image>
             <format>L8</format>
-            <width>640</width>
-            <height>480</height>
+            <width>${width}</width>
+            <height>${height}</height>
           </image>
           <clip>
-            <near>0.01</near>
+            <near>${min_range}</near>
             <far>${max_range}</far>
           </clip>
@@ -666,5 +666,5 @@
   </xacro:macro>
   <!-- VI-Sensor Macro -->
-  <xacro:macro name="vi_sensor_macro" params="namespace parent_link enable_cameras enable_depth enable_ground_truth horizontal_fov *origin">
+  <xacro:macro name="vi_sensor_macro" params="namespace parent_link enable_cameras enable_depth enable_ground_truth horizontal_fov stereo_frame_rate stereo_max_range stereo_min_range stereo_width stereo_height depth_frame_rate depth_max_range depth_min_range depth_width depth_height *origin">
     <!-- Vi Sensor Link -->
     <link name="${namespace}/vi_sensor_link">
@@ -697,6 +697,6 @@
       <xacro:vi_sensor_stereo_camera_macro
         namespace="${namespace}" parent_link="${namespace}/vi_sensor_link"
-        frame_rate="30.0" origin_offset_x="0.015" baseline_y="${0.055*2}"
-        origin_offset_z="0.0065" max_range="30.0" horizontal_fov="${horizontal_fov}">
+        frame_rate="${stereo_frame_rate}" origin_offset_x="0.015" baseline_y="${0.055*2}"
+        origin_offset_z="0.0065" max_range="${stereo_max_range}" min_range="${stereo_min_range}" width="${stereo_width}" height="${stereo_height}" horizontal_fov="${horizontal_fov}">
       </xacro:vi_sensor_stereo_camera_macro>
     </xacro:if>
@@ -705,5 +705,5 @@
       <xacro:vi_sensor_depth_macro
         namespace="${namespace}" parent_link="${namespace}/vi_sensor_link"
-        camera_suffix="depth" frame_rate="30.0" max_range="10.0" horizontal_fov="${horizontal_fov}">
+        camera_suffix="depth" frame_rate="${depth_frame_rate}" max_range="${depth_max_range}" min_range="${depth_min_range}" width="${depth_width}" height="${depth_height}" horizontal_fov="${horizontal_fov}">
         <origin xyz="0.015 0.055 0.0065" rpy="0 0 0" />
       </xacro:vi_sensor_depth_macro>

File: rotors_description/urdf/firefly_base.xacro (robot description, xacro)
@@ -47,5 +47,5 @@
   <!-- gimbal-->
   <gimbal namespace="${namespace}" parent="${namespace}/base_link"/>
-  <!-- depth camera-->
+  <!-- vi_sensor-->
   <vi_sensor_macro
     namespace="${namespace}/vi_sensor"
@@ -54,5 +54,15 @@
     enable_depth="true"
     enable_ground_truth="true"
-    horizontal_fov="$(arg horizontal_fov)">
+    horizontal_fov="$(arg horizontal_fov)"
+    depth_frame_rate="$(arg depth_frame_rate)"
+    depth_max_range="$(arg depth_max_range)"
+    depth_min_range="$(arg depth_min_range)"
+    depth_width="$(arg depth_width)"
+    depth_height="$(arg depth_height)"
+    stereo_frame_rate="$(arg stereo_frame_rate)"
+    stereo_max_range="$(arg stereo_max_range)"
+    stereo_min_range="$(arg stereo_min_range)"
+    stereo_width="$(arg stereo_width)"
+    stereo_height="$(arg stereo_height)">
     <origin xyz="0 0 0" rpy="0.0 0.1 0.0" />
 </vi_sensor_macro>
